Commit message: The joint between the laser and the volksbot can now be controlled. The simulation does not work too well right now.

File: volksbot_sim/urdf/volksbot_las_lev.urdf.xacro (robot description, xacro)
@@ -553,10 +553,10 @@
 	</link>
 <!--position laser_platform-->
-	<joint name="base_link_to_laser_platform" type="revolute">
+	<joint name="base_link_to_laser_platform" type="continuous">   <!--revolute-->
 	<!--<joint name="base_link_to_laser_platform" type="fixed">-->
 		<parent link="base_link"/>
 		<child link="laser_platform"/>
 		 <axis xyz="1 0 0"/>
-		 <limit effort="1000.0" lower="0.0" upper="0.548" velocity="0.5"/>
+		 <!--<limit effort="1000.0" lower="0.0" upper="0.548" velocity="0.5"/>-->
 		<origin rpy="0 0 0" xyz="0 0 0.405"/>
 	</joint>
@@ -650,5 +650,6 @@
 <!--  ############################  Husky Controller Fuerte  ###################################-->
 <gazebo>
-			<controller:husky_plugin name="husky_diff_controller" plugin="libhusky_description_new.so">
+	<!--		<controller:husky_plugin name="husky_diff_controller" plugin="libhusky_description_new.so"> -->
+				<controller:husky_plugin name="husky_diff_controller" plugin="libhusky_description_new_exp.so">
 		        <alwaysOn>true</alwaysOn>
 		        <updateRate>100.0</updateRate>  <!-- alt 100 -->

Commit message: Added a second moveable joint in order to tilt the laser. The only thing that has to be implemented is a PI or a PID controller to level the laser.

File: volksbot_sim/urdf/volksbot_las_lev.urdf.xacro (robot description, xacro)
@@ -530,4 +530,30 @@
   </gazebo>
 <!--  ###############################  laser ######################################### -->
+	<link name="roll_tilt_base">
+		<visual>
+			<geometry>
+				<box size="0.001 0.001 0.001"/>
+			</geometry>
+			<origin rpy="0 0 0" xyz="0 0 0"/>
+		</visual>
+	<!--	<collision>
+			<geometry>
+				<box size="0.001 0.001 0.001"/>
+			</geometry>
+			<origin xyz="0 0 0"/>
+		</collision>-->
+		<inertial>
+			<mass value="0.01"/>
+			<inertia ixx=".001" ixy="0.0" ixz="0.0" iyy=".001" iyz="0.0" izz=".001"/>
+			<origin xyz="0 0 0.0" />
+		</inertial>
+	</link>
+	<joint name="base_link_to_roll_tilt_base" type="continuous">   <!--revolute-->
+		<parent link="base_link"/>
+		<child link="roll_tilt_base"/>
+		 <axis xyz="1 0 0"/>
+		 <!--<limit effort="1000.0" lower="0.0" upper="0.548" velocity="0.5"/>-->
+		<origin rpy="0 0 0" xyz="0 0 0.405"/>
+	</joint>
 	<link name="laser_platform">
 		<visual>
@@ -553,11 +579,11 @@
 	</link>
 <!--position laser_platform-->
-	<joint name="base_link_to_laser_platform" type="continuous">   <!--revolute-->
+	<joint name="roll_tilt_base_to_laser_platform" type="continuous">   <!--revolute-->
 	<!--<joint name="base_link_to_laser_platform" type="fixed">-->
-		<parent link="base_link"/>
+		<parent link="roll_tilt_base"/>
 		<child link="laser_platform"/>
-		 <axis xyz="1 0 0"/>
+		 <axis xyz="0 1 0"/>
 		 <!--<limit effort="1000.0" lower="0.0" upper="0.548" velocity="0.5"/>-->
-		<origin rpy="0 0 0" xyz="0 0 0.405"/>
+		<origin rpy="0 0 0" xyz="0 0 0"/>
 	</joint>
 	<gazebo reference="platform">

Commit message: Changed the urdf so the laser tf frame fits the normal robot configuration.

File: volksbot_sim/urdf/volksbot_las_lev.urdf.xacro (robot description, xacro)
@@ -625,7 +625,9 @@
     <origin rpy="0 0 0" xyz="0 0 0.05"/>
     <parent link="laser_base_link"/>
-    <child link="base_scan_link"/>
+    <!--<child link="base_scan_link"/>-->
+    <child link="laser"/>
   </joint>
-  <link name="base_scan_link" type="laser">
+  <!--<link name="base_scan_link" type="laser">-->
+  <link name="laser" type="laser">
     <inertial>
       <mass value="0.1"/>
@@ -646,9 +648,11 @@
     </collision>
   </link>
-  <gazebo reference="base_scan_link">
+  <!--<gazebo reference="base_scan_link">-->
+  <gazebo reference="laser">
     <material>Gazebo/Black</material>
   </gazebo>
 <!--Laserscanner Einstellungen-->
-  <gazebo reference="base_scan_link">
+  <!--<gazebo reference="base_scan_link">-->
+  <gazebo reference="laser">
     <sensor:ray name="laser">
       <rayCount>683</rayCount>
